File: osw-light.kicad_pcb (KiCad board)
At the start: 4 copper layers, 36.1 x 36.1 mm, 55 parts, among them J1 Conn_01x02, Q1 2N7002, SW1 SW_Push, SW2 SW_Push, SW4 SW_Push, SW5 SW_Push, U1 DS3231MZ, U10 XC6209, U11 MCP73831T-2ACI_OT, U13 XC6209, U2 BMA400, U4 GC9A01_IPS_display, U5 USB-OTG, U6 CH340E, U7 ttgo-32-micro, U9 TPS2115A

Commit message: first commit + CAD models
Added CAD files for V1 nixie watch, this includes
- chassis
- lid
- 1.25 mm acrylic pane
- IN 16 nixie tubes
- Daughter board PCB
- Master PCB space claim
Other:
- net class Default removed
